Commit message: feat: add landing gear to URDF model

File: bpla_description/urdf/quadcopter.urdf (robot description, URDF)
Before this commit: robot quadcopter, 13 links, 12 joints
Links:
- added link landing_gear_front; visual cylinder length=0.1 radius=0.005
- added link landing_gear_rear; visual cylinder length=0.1 radius=0.005
Joints:
- added joint lg_front_joint: type fixed, parent base_link, child landing_gear_front, origin xyz=0 0.08 -0.03 rpy=0 1.5708 0
- added joint lg_rear_joint: type fixed, parent base_link, child landing_gear_rear, origin xyz=0 -0.08 -0.03 rpy=0 1.5708 0
